File: pcb/blimpy.brd (EAGLE design)
At the start: 70 x 70 mm, 74 parts, among them J4 3-PIN SMD, J5 3-PIN SMD, J6 3-PIN SMD, J7 3-PIN SMD, Q1 mmbt2222, Q2 mmbt2222, Q3 DMG3415U, U1 RGB, U10 MAX17048, U2 AP2112-3.3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

Commit message: small fix
Routing:
- net V_USB: track 24.2 -> 25.7 mm
Changed lines of the file:
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@@
 <wire x1="10.65" y1="26.2" x2="10.85" y2="26" width="0.4" layer="1"/>
 <wire x1="10.85" y1="26" x2="13.15" y2="26" width="0.4" layer="1"/>
-<wire x1="5" y1="44.5" x2="5" y2="46" width="0" layer="19" extent="1-1"/>
+<wire x1="5" y1="44.5" x2="5" y2="46" width="0.4" layer="1"/>
 <wire x1="13" y1="30.95" x2="15" y2="43" width="0" layer="19" extent="1-1"/>
 <wire x1="13.15" y1="26" x2="13" y2="30.95" width="0" layer="19" extent="1-1"/>
-<wire x1="-7" y1="35.5936" x2="5" y2="44.5" width="0" layer="19" extent="1-1"/>
+<wire x1="-7" y1="35.5936" x2="5" y2="46" width="0" layer="19" extent="1-1"/>
 <wire x1="-7.85" y1="33.5" x2="-7" y2="35.5936" width="0" layer="19" extent="1-1"/>
 <wire x1="-9.6999" y1="35.05" x2="-7.85" y2="33.5" width="0" layer="19" extent="1-1"/>

Commit message: updated
Parts:
- moved D2 5.70 mm to (-14.5, 36.0), turned to 0 degrees
- moved C3 0.50 mm to (-11.0, 33.0)
Changed lines of the file:
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@@
 </element>
 <element name="U3" library="microbuilder" package="SOT23-5" value="MCP73831T-2" x="-11" y="36" smashed="yes" rot="R270">
-<attribute name="NAME" x="-10.478" y="34" size="0.6" layer="25" font="vector" ratio="15" rot="R180"/>
-</element>
-<element name="D2" library="microbuilder" package="CHIPLED_0805_NOOUTLINE" value="ORANGE" x="-11" y="40.5" smashed="yes" rot="R270">
-<attribute name="NAME" x="-11" y="39.5" size="0.6" layer="25" font="vector" ratio="15" rot="R180" align="bottom-center"/>
+<attribute name="NAME" x="-9.022" y="36" size="0.6" layer="25" font="vector" ratio="15"/>
+</element>
+<element name="D2" library="microbuilder" package="CHIPLED_0805_NOOUTLINE" value="ORANGE" x="-14.5" y="36" smashed="yes">
+<attribute name="NAME" x="-15.5" y="36" size="0.6" layer="25" font="vector" ratio="15" rot="R90" align="bottom-center"/>
 </element>
 <element name="R2" library="SparkFun-Resistors" package="0603" value="1k" x="-11" y="39" smashed="yes">
@@
 <attribute name="VALUE" value="1k" x="-11" y="39" size="1.778" layer="27" display="off"/>
 </element>
-<element name="C3" library="SparkFun-Capacitors" package="0603" value="10uF" x="-11" y="32.5" smashed="yes">
-<attribute name="NAME" x="-11" y="33.5" size="0.6" layer="25" font="vector" ratio="15" align="bottom-center"/>
-<attribute name="PROD_ID" value="CAP-11015" x="-11" y="32.5" size="1.778" layer="27" display="off"/>
+<element name="C3" library="SparkFun-Capacitors" package="0603" value="10uF" x="-11" y="33" smashed="yes">
+<attribute name="NAME" x="-11" y="32" size="0.6" layer="25" font="vector" ratio="15" rot="R180" align="bottom-center"/>
+<attribute name="PROD_ID" value="CAP-11015" x="-11" y="33" size="1.778" layer="27" display="off"/>
 </element>
 <element name="U7" library="microbuilder" package="QFN24_4MM_SMSC" value="CP2104" x="12.5" y="46" smashed="yes">
@@
 </element>
 <element name="R4" library="SparkFun-Resistors" library_urn="urn:adsk.eagle:library:532" package="0603" package3d_urn="urn:adsk.eagle:package:39650/1" value="2.0k" x="-7" y="38.5" smashed="yes" rot="R180">
-<attribute name="NAME" x="-9" y="38.5" size="0.6" layer="25" font="vector" ratio="15" rot="R90" align="bottom-center"/>
+<attribute name="NAME" x="-7" y="39.5" size="0.6" layer="25" font="vector" ratio="15" align="bottom-center"/>
 <attribute name="PROD_ID" value="RES-08296" x="-7" y="38.5" size="1.778" layer="27" rot="R180" display="off"/>
 </element>
@@
 </element>
 <element name="C9" library="SparkFun-Capacitors" package="0603" value="10uF" x="-7" y="33.5" smashed="yes">
-<attribute name="NAME" x="-7" y="34.5" size="0.6" layer="25" font="vector" ratio="15" align="bottom-center"/>
+<attribute name="NAME" x="-7" y="32.5" size="0.6" layer="25" font="vector" ratio="15" rot="R180" align="bottom-center"/>
 <attribute name="PROD_ID" value="CAP-11015" x="-7" y="33.5" size="1.778" layer="27" display="off"/>
 </element>
@@
 <wire x1="-6.15" y1="38.5" x2="7" y2="42.775" width="0" layer="19" extent="1-1"/>
 <wire x1="-6.15" y1="33.5" x2="-6.15" y2="38.5" width="0" layer="19" extent="1-1"/>
-<wire x1="-10.15" y1="32.5" x2="-6.15" y2="33.5" width="0" layer="19" extent="1-1"/>
-<wire x1="-12.3001" y1="36" x2="-10.15" y2="32.5" width="0" layer="19" extent="1-1"/>
+<wire x1="-10.15" y1="33" x2="-6.15" y2="33.5" width="0" layer="19" extent="1-1"/>
+<wire x1="-12.3001" y1="36" x2="-10.15" y2="33" width="0" layer="19" extent="1-1"/>
 <wire x1="-8.75" y1="46.51" x2="-6.15" y2="38.5" width="0" layer="19" extent="1-1"/>
 <wire x1="-9.5" y1="47.5" x2="-8.75" y2="46.51" width="0" layer="19" extent="1-1"/>
@@
 <contactref element="D2" pad="C"/>
 <contactref element="R2" pad="1"/>
-<wire x1="-11.85" y1="39" x2="-9.95" y2="40.5" width="0" layer="19" extent="1-1"/>
+<wire x1="-11.85" y1="39" x2="-14.5" y2="37.05" width="0" layer="19" extent="1-1"/>
 </signal>
 <signal name="N$3">
@@
 <wire x1="-7.85" y1="33.5" x2="-7" y2="35.5936" width="0" layer="19" extent="1-1"/>
 <wire x1="-9.6999" y1="35.05" x2="-7.85" y2="33.5" width="0" layer="19" extent="1-1"/>
-<wire x1="-12.05" y1="40.5" x2="-9.6999" y2="35.05" width="0" layer="19" extent="1-1"/>
+<wire x1="-14.5" y1="34.95" x2="-9.6999" y2="35.05" width="0" layer="19" extent="1-1"/>
 </signal>
 <signal name="V_BATT">
@@
 <wire x1="-9.75" y1="46.51" x2="-9.25" y2="46.51" width="0" layer="19" extent="1-1"/>
 <wire x1="-12.3001" y1="35.05" x2="-9.75" y2="46.51" width="0" layer="19" extent="1-1"/>
-<wire x1="-11.85" y1="32.5" x2="-12.3001" y2="35.05" width="0" layer="19" extent="1-1"/>
+<wire x1="-11.85" y1="33" x2="-12.3001" y2="35.05" width="0" layer="19" extent="1-1"/>
 <wire x1="6.51" y1="61.73" x2="-7" y2="46.65" width="0" layer="19" extent="1-1"/>
 <wire x1="63.49" y1="8.27" x2="48.575" y2="22.125" width="0" layer="19" extent="1-1"/>

Commit message: connect imu
Routing:
- net 3.3V: track 115.1 -> 130.0 mm
- net IMU_RST: track 0.00 -> 4.61 mm
- net IMU_INT: track 0.00 -> 3.40 mm
- net N$14: track 0.00 -> 3.27 mm
- net N$15: track 0.00 -> 2.69 mm
- net N$16: track 0.00 -> 2.47 mm
- net IMU_BOOT: track 0.00 -> 2.35 mm
- net SCL: track 9.48 -> 11.7 mm
- net SDA: track 9.65 -> 11.1 mm
- net V_BATT: vias 0 -> 1
Changed lines of the file:
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@@
 <contactref element="D2" pad="C"/>
 <contactref element="R2" pad="1"/>
-<wire x1="-11.85" y1="39" x2="-14.5" y2="37.05" width="0" layer="19" extent="1-1"/>
+<wire x1="-14.5" y1="37.05" x2="-11.85" y2="39" width="0" layer="19" extent="1-1"/>
 </signal>
 <signal name="N$3">
@@
 <wire x1="67" y1="52" x2="66.65" y2="52.35" width="0.2" layer="1"/>
 <wire x1="66.65" y1="52.35" x2="66" y2="52.35" width="0.2" layer="1"/>
+<wire x1="30.5" y1="35.85" x2="31.15" y2="35.85" width="0.2" layer="1"/>
+<wire x1="31.75" y1="35.25" x2="32.6" y2="35.25" width="0.2" layer="1"/>
+<wire x1="31.15" y1="35.85" x2="31.75" y2="35.25" width="0.2" layer="1"/>
+<wire x1="41.35" y1="34" x2="41.35" y2="36" width="0.2" layer="1"/>
+<wire x1="34.75" y1="33.3" x2="34.75" y2="32.25" width="0.2" layer="1"/>
+<wire x1="36.15" y1="31" x2="35.5" y2="31" width="0.2" layer="1"/>
+<wire x1="35.5" y1="31" x2="35" y2="31.5" width="0.2" layer="1"/>
+<wire x1="35" y1="31.5" x2="35" y2="32" width="0.2" layer="1"/>
+<wire x1="35" y1="32" x2="34.75" y2="32.25" width="0.2" layer="1"/>
+<wire x1="33.25" y1="36.7" x2="33.25" y2="37.6" width="0.2" layer="1"/>
+<wire x1="33.25" y1="37.6" x2="34.15" y2="38.5" width="0.2" layer="1"/>
+<wire x1="33.25" y1="36.7" x2="33.25" y2="36.21805" width="0.2" layer="1"/>
+<wire x1="33.75" y1="35.25" x2="33.5" y2="35.25" width="0.2" layer="1"/>
+<wire x1="33.5" y1="35.25" x2="32.6" y2="35.25" width="0.2" layer="1"/>
+<wire x1="33.25" y1="36.21805" x2="33.5" y2="35.96805" width="0.2" layer="1"/>
+<wire x1="34.75" y1="33.3" x2="34.75" y2="34.25" width="0.2" layer="1"/>
+<wire x1="34.75" y1="34.25" x2="33.75" y2="35.25" width="0.2" layer="1"/>
+<wire x1="33.5" y1="35.96805" x2="33.5" y2="35.25" width="0.2" layer="1"/>
 <wire x1="45.975" y1="47.875" x2="66" y2="52.35" width="0" layer="19" extent="1-1"/>
 <wire x1="34.15" y1="38.5" x2="33.025" y2="44.5" width="0" layer="19" extent="1-1"/>
-<wire x1="33.25" y1="36.7" x2="34.15" y2="38.5" width="0" layer="19" extent="1-1"/>
-<wire x1="32.6" y1="35.25" x2="33.25" y2="36.7" width="0" layer="19" extent="1-1"/>
-<wire x1="30.5" y1="35.85" x2="32.6" y2="35.25" width="0" layer="19" extent="1-1"/>
-<wire x1="34.75" y1="33.3" x2="32.6" y2="35.25" width="0" layer="19" extent="1-1"/>
-<wire x1="36.15" y1="31" x2="34.75" y2="33.3" width="0" layer="19" extent="1-1"/>
 <wire x1="34.5" y1="29.5" x2="36.15" y2="31" width="0" layer="19" extent="1-1"/>
 <wire x1="33.025" y1="25.5" x2="34.6" y2="27.475" width="0" layer="19" extent="1-1"/>
 <wire x1="36.975" y1="25.5" x2="34.6" y2="27.475" width="0" layer="19" extent="1-1"/>
 <wire x1="41.35" y1="34" x2="36.15" y2="31" width="0" layer="19" extent="1-1"/>
-<wire x1="41.35" y1="36" x2="41.35" y2="34" width="0" layer="19" extent="1-1"/>
 <wire x1="13.15" y1="21.5" x2="24.025" y2="22.125" width="0" layer="19" extent="1-1"/>
 <wire x1="11.25" y1="44" x2="25.325" y2="47.875" width="0" layer="19" extent="1-1"/>
@@
 <wire x1="61.73" y1="26.26" x2="61.73" y2="21.12" width="0.2" layer="1"/>
 <wire x1="61.73" y1="21.12" x2="62" y2="20.85" width="0.2" layer="1"/>
+<wire x1="37.25" y1="36.7" x2="37.25" y2="37.75" width="0.2" layer="1"/>
+<wire x1="37.25" y1="37.75" x2="37.5" y2="38" width="0.2" layer="1"/>
 <wire x1="35.4" y1="27.475" x2="61.73" y2="26.26" width="0" layer="19" extent="1-1"/>
 <wire x1="37.25" y1="36.7" x2="35.5" y2="29.5" width="0" layer="19" extent="1-1"/>
-<wire x1="34.5" y1="40.5" x2="37.25" y2="36.7" width="0" layer="19" extent="1-1"/>
+<wire x1="34.5" y1="40.5" x2="37.5" y2="38" width="0" layer="19" extent="1-1"/>
 <wire x1="-10.25" y1="48.49" x2="34.6" y2="42.525" width="0" layer="19" extent="1-1"/>
 </signal>
@@
 <wire x1="65.54" y1="26.26" x2="65.54" y2="20.89" width="0.2" layer="1"/>
 <wire x1="65.54" y1="20.89" x2="65.5" y2="20.85" width="0.2" layer="1"/>
-<wire x1="37.4" y1="35.75" x2="65.54" y2="26.26" width="0" layer="19" extent="1-1"/>
-<wire x1="35" y1="40.5" x2="37.4" y2="35.75" width="0" layer="19" extent="1-1"/>
+<wire x1="37.4" y1="35.75" x2="38.25" y2="35.75" width="0.2" layer="1"/>
+<wire x1="38.25" y1="35.75" x2="38.5" y2="36" width="0.2" layer="1"/>
+<wire x1="38.5" y1="36" x2="38.5" y2="37" width="0.2" layer="1"/>
+<wire x1="38.5" y1="37" x2="65.54" y2="26.26" width="0" layer="19" extent="1-1"/>
+<wire x1="35" y1="40.5" x2="38.5" y2="37" width="0" layer="19" extent="1-1"/>
 <wire x1="35" y1="29.5" x2="37.4" y2="35.75" width="0" layer="19" extent="1-1"/>
 <wire x1="-9.75" y1="48.49" x2="35" y2="42.525" width="0" layer="19" extent="1-1"/>
@@
 <signal name="IMU_INT">
 <contactref element="U4" pad="14"/>
+<wire x1="36.75" y1="33.3" x2="36.75" y2="32.75" width="0.2" layer="1"/>
+<wire x1="36.75" y1="32.75" x2="37" y2="32.5" width="0.2" layer="1"/>
+<wire x1="37" y1="32.5" x2="39.5" y2="32.5" width="0.2" layer="1"/>
 </signal>
 <signal name="IMU_BOOT">
 <contactref element="U4" pad="4"/>
 <contactref element="R16" pad="1"/>
-<wire x1="30.5" y1="34.15" x2="32.6" y2="34.75" width="0" layer="19" extent="1-1"/>
+<wire x1="30.5" y1="34.15" x2="31.15" y2="34.15" width="0.2" layer="1"/>
+<wire x1="31.75" y1="34.75" x2="32.6" y2="34.75" width="0.2" layer="1"/>
+<wire x1="31.15" y1="34.15" x2="31.75" y2="34.75" width="0.2" layer="1"/>
 </signal>
 <signal name="IMU_RST">
 <contactref element="U4" pad="11"/>
+<wire x1="35.25" y1="33.3" x2="35.25" y2="32.75" width="0.2" layer="1"/>
+<wire x1="35.25" y1="32.75" x2="36" y2="32" width="0.2" layer="1"/>
+<wire x1="36" y1="32" x2="39" y2="32" width="0.2" layer="1"/>
 </signal>
 <signal name="N$14">
 <contactref element="U4" pad="16"/>
 <contactref element="R8" pad="1"/>
-<wire x1="37.4" y1="34.25" x2="39.65" y2="36" width="0" layer="19" extent="1-1"/>
+<wire x1="37.4" y1="34.25" x2="38.25" y2="34.25" width="0.2" layer="1"/>
+<wire x1="38.25" y1="34.25" x2="38.5" y2="34.5" width="0.2" layer="1"/>
+<wire x1="38.5" y1="34.5" x2="38.5" y2="35" width="0.2" layer="1"/>
+<wire x1="38.5" y1="35" x2="39.5" y2="36" width="0.2" layer="1"/>
+<wire x1="39.5" y1="36" x2="39.65" y2="36" width="0.2" layer="1"/>
 </signal>
 <signal name="N$15">
 <contactref element="U4" pad="15"/>
 <contactref element="R15" pad="1"/>
-<wire x1="37.25" y1="33.3" x2="39.65" y2="34" width="0" layer="19" extent="1-1"/>
+<wire x1="37.25" y1="33.3" x2="38.3" y2="33.3" width="0.2" layer="1"/>
+<wire x1="39" y1="34" x2="39.65" y2="34" width="0.2" layer="1"/>
+<wire x1="38.3" y1="33.3" x2="39" y2="34" width="0.2" layer="1"/>
 </signal>
 <signal name="N$16">
 <contactref element="U4" pad="9"/>
 <contactref element="C1" pad="1"/>
-<wire x1="33.85" y1="31" x2="34.25" y2="33.3" width="0" layer="19" extent="1-1"/>
+<wire x1="34.25" y1="33.3" x2="34.25" y2="32.25" width="0.2" layer="1"/>
+<wire x1="33.85" y1="31.85" x2="33.85" y2="31" width="0.2" layer="1"/>
+<wire x1="34.25" y1="32.25" x2="33.85" y2="31.85" width="0.2" layer="1"/>
 </signal>
 <signal name="IO2_RST">
@@
 <wire x1="-14.5" y1="34.95" x2="-9.6999" y2="35.05" width="0" layer="19" extent="1-1"/>
 </signal>
-<signal name="V_BATT">
+<signal name="V_BATT" airwireshidden="yes">
 <contactref element="Q3" pad="3"/>
 <contactref element="U3" pad="3"/>
@@
 <wire x1="34" y1="18.85" x2="36" y2="18.85" width="1.2" layer="1"/>
 <wire x1="8.2" y1="36" x2="12.5" y2="36" width="0.8" layer="1"/>
+<via x="61.5" y="3.5" extent="1-16" drill="0.4"/>
 <wire x1="48.575" y1="47.875" x2="59.51" y2="61.73" width="0" layer="19" extent="1-1"/>
 <wire x1="12.5" y1="36" x2="21.425" y2="47.875" width="0" layer="19" extent="1-1"/>
@@
 <wire x1="6.51" y1="61.73" x2="-7" y2="46.65" width="0" layer="19" extent="1-1"/>
 <wire x1="63.49" y1="8.27" x2="48.575" y2="22.125" width="0" layer="19" extent="1-1"/>
+<wire x1="61.5" y1="3.5" x2="63.49" y2="8.27" width="0" layer="19" extent="1-1"/>
 </signal>
 <signal name="HB1-A1">

Commit message: more traces
Parts:
- moved C3 33.0 mm to (22.0, 32.0)
- moved C9 33.0 mm to (26.0, 32.5)
- moved D2 33.0 mm to (18.5, 35.0)
- moved JP1 33.0 mm to (26.0, 35.0)
- moved R2 33.0 mm to (22.0, 38.0)
- moved R4 33.0 mm to (26.0, 37.5)
- moved U3 33.0 mm to (22.0, 35.0)
- moved U10 26.9 mm to (14.0, 34.5)
- moved C11 22.8 mm to (14.0, 38.5), turned to 0 degrees
- moved C2 1.50 mm to (14.0, 42.0)
- moved U7 1.50 mm to (14.0, 46.0)
- moved R1 1.00 mm to (10.0, 49.5)
- moved R3 1.00 mm to (10.0, 42.5)
- moved J1 0.50 mm to (7.50, 46.0)
Routing:
- net V_USB: track 25.7 -> 31.4 mm
- net N$4: track 0.00 -> 5.14 mm
- net N$1: track 0.00 -> 4.01 mm
- net N$3: track 0.00 -> 3.38 mm
- net V_BATT: track 87.2 -> 85.1 mm
- net N$6: track 8.14 -> 9.14 mm
- net N$2: track 5.35 -> 6.35 mm
- net N$5: track 2.96 -> 3.46 mm
- net N$17: track 2.37 -> 2.87 mm

Commit message: show all
Routing:
- net GND: track 136.9 -> 138.0 mm
Changed lines of the file:
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@@
 <wire x1="24.675" y1="44.825" x2="25" y2="44.5" width="0.2" layer="1"/>
 <via x="25" y="44.5" extent="1-16" drill="0.3"/>
-<wire x1="35.85" y1="48.5" x2="38.5" y2="48.5" width="0.2" layer="1"/>
-<wire x1="38.5" y1="48.5" x2="39" y2="48" width="0.2" layer="1"/>
+<wire x1="35.85" y1="48.5" x2="37.675" y2="46.675" width="0.2" layer="1"/>
+<wire x1="39" y1="48" x2="37.675" y2="46.675" width="0.2" layer="1"/>
 <via x="39" y="48" extent="1-16" drill="0.3"/>
 <wire x1="35.4" y1="42.525" x2="35.4" y2="40.6" width="0.2" layer="1"/>
@@
 <wire x1="33.95" y1="52.9" x2="34" y2="52.85" width="0" layer="19" extent="1-1"/>
 <wire x1="36" y1="52.85" x2="34" y2="52.85" width="0" layer="19" extent="1-1"/>
-<wire x1="35.85" y1="48.5" x2="36" y2="52.85" width="0" layer="19" extent="1-1"/>
+<wire x1="39" y1="48" x2="36" y2="52.85" width="0" layer="19" extent="1-1"/>
 <wire x1="35.85" y1="38.5" x2="35.5" y2="40.5" width="0" layer="19" extent="1-1"/>
 <wire x1="34.75" y1="36.7" x2="35.85" y2="38.5" width="0" layer="19" extent="1-1"/>
@@
 <wire x1="26" y1="36" x2="25.15" y2="36.85" width="0.2" layer="1"/>
 </signal>
-<signal name="3.3V" airwireshidden="yes">
+<signal name="3.3V">
 <contactref element="HB4" pad="20"/>
 <contactref element="HB4" pad="19"/>
@@
 <wire x1="16.5" y1="43" x2="18.5" y2="33.95" width="0" layer="19" extent="1-1"/>
 </signal>
-<signal name="V_BATT" airwireshidden="yes">
+<signal name="V_BATT">
 <contactref element="Q3" pad="3"/>
 <contactref element="U3" pad="3"/>

Commit message: small fixes
Changed lines of the file:
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@@
 </element>
 <element name="U3" library="microbuilder" package="SOT23-5" value="MCP73831T-2" x="22" y="35" smashed="yes" rot="R270">
-<attribute name="NAME" x="23.978" y="35" size="0.6" layer="25" font="vector" ratio="15"/>
+<attribute name="NAME" x="23.478" y="35" size="0.6" layer="25" font="vector" ratio="15" align="center-left"/>
 </element>
 <element name="D2" library="microbuilder" package="CHIPLED_0805_NOOUTLINE" value="ORANGE" x="18.5" y="35" smashed="yes">
@@
 </element>
 <element name="Q1" library="SparkFun" package="SOT23-3" value="mmbt2222" x="59" y="53.5" smashed="yes">
-<attribute name="NAME" x="57.5" y="54.5" size="0.6" layer="25" font="vector" ratio="15"/>
+<attribute name="NAME" x="57" y="54" size="0.6" layer="25" font="vector" ratio="15" rot="R180"/>
 </element>
 <element name="Q2" library="SparkFun" package="SOT23-3" value="mmbt2222" x="59" y="49.5" smashed="yes" rot="R180">
-<attribute name="NAME" x="60.5" y="48.5" size="0.6" layer="25" font="vector" ratio="15" rot="R180"/>
+<attribute name="NAME" x="61" y="49" size="0.6" layer="25" font="vector" ratio="15"/>
 </element>
 <element name="Q3" library="microbuilder" package="SOT23-R" value="DMG3415U" x="14" y="30" smashed="yes" rot="R270">
@@
 </element>
 <element name="S1" library="SparkFun-Switches" package="SWITCH_SPST_SMD_A" value="PWR" x="2.5" y="24.5" smashed="yes" rot="R90">
-<attribute name="NAME" x="5" y="25" size="0.6" layer="25" font="vector" ratio="15" align="bottom-center"/>
+<attribute name="NAME" x="4.5" y="25" size="0.6" layer="25" font="vector" ratio="15"/>
 <attribute name="PROD_ID" value="SWCH-10651" x="2.5" y="24.5" size="1.778" layer="27" rot="R90" display="off"/>
 <attribute name="SF_SKU" value="COM-10860" x="2.5" y="24.5" size="1.778" layer="27" rot="R90" display="off"/>
@@
 </element>
 <element name="C4" library="SparkFun-Capacitors" package="0603" value="0.1uF" x="37" y="31" smashed="yes">
-<attribute name="NAME" x="37" y="32" size="0.6" layer="25" font="vector" ratio="15" align="bottom-center"/>
+<attribute name="NAME" x="37" y="30" size="0.6" layer="25" font="vector" ratio="15" rot="R180" align="bottom-center"/>
 <attribute name="PROD_ID" value="CAP-08604" x="37" y="31" size="1.778" layer="27" display="off"/>
 </element>
 <element name="C10" library="SparkFun-Capacitors" package="0603" value="0.1uF" x="35" y="38.5" smashed="yes">
-<attribute name="NAME" x="33" y="38.5" size="0.6" layer="25" font="vector" ratio="15" rot="R90" align="bottom-center"/>
+<attribute name="NAME" x="35" y="39.5" size="0.6" layer="25" font="vector" ratio="15" align="bottom-center"/>
 <attribute name="PROD_ID" value="CAP-08604" x="35" y="38.5" size="1.778" layer="27" display="off"/>
 </element>
@@
 </element>
 <element name="R10" library="SparkFun-Resistors" package="0603" value="10k" x="56.5" y="51.5" smashed="yes" rot="R90">
-<attribute name="NAME" x="55.5" y="51.5" size="0.6" layer="25" font="vector" ratio="15" rot="R90" align="bottom-center"/>
+<attribute name="NAME" x="56.5" y="49.5" size="0.6" layer="25" font="vector" ratio="15" rot="R180" align="bottom-center"/>
 <attribute name="PROD_ID" value="RES-00824" x="56.5" y="51.5" size="1.778" layer="27" rot="R90" display="off"/>
 </element>
@@
 </element>
 <element name="U4" library="BNO080" package="LGA-28" value="BNO080" x="35" y="35" smashed="yes" rot="R90">
-<attribute name="NAME" x="32" y="37.5" size="0.6" layer="25" font="vector" ratio="15"/>
+<attribute name="NAME" x="32" y="37.5" size="0.6" layer="25" font="vector" ratio="15" align="bottom-right"/>
 </element>
 <element name="R8" library="SparkFun-Resistors" package="0603" value="4.7k" x="40.5" y="36" smashed="yes">
@@
 </element>
 <element name="J2" library="SparkFun-Connectors" library_urn="urn:adsk.eagle:library:513" package="JST-2-SMD" package3d_urn="urn:adsk.eagle:package:38042/1" value="" x="4.5" y="35" smashed="yes" rot="R90">
-<attribute name="NAME" x="9.5" y="38" size="0.6" layer="25" font="vector" ratio="15"/>
+<attribute name="NAME" x="9.5" y="38.5" size="0.6" layer="25" font="vector" ratio="15" align="center-left"/>
 <attribute name="PROD_ID" value="CONN-11443" x="4.5" y="35" size="1.778" layer="27" rot="R90" display="off"/>
 <attribute name="VALUE" x="3.865" y="33.349" size="0.6096" layer="27" font="vector" ratio="20" rot="R90"/>
@@
 <wire x1="33.95" y1="52.9" x2="34" y2="52.85" width="0" layer="19" extent="1-1"/>
 <wire x1="36" y1="52.85" x2="34" y2="52.85" width="0" layer="19" extent="1-1"/>
-<wire x1="39" y1="48" x2="36" y2="52.85" width="0" layer="19" extent="1-1"/>
+<wire x1="35.85" y1="48.5" x2="36" y2="52.85" width="0" layer="19" extent="1-1"/>
 <wire x1="35.85" y1="38.5" x2="35.5" y2="40.5" width="0" layer="19" extent="1-1"/>
 <wire x1="34.75" y1="36.7" x2="35.85" y2="38.5" width="0" layer="19" extent="1-1"/>
@@
 <contactref element="U7" pad="4"/>
 <via x="10" y="47" extent="1-16" drill="0.3"/>
-<via x="10" y="45.3436" extent="1-16" drill="0.3"/>
-<wire x1="10" y1="45.3436" x2="10.4064" y2="45.75" width="0.2" layer="1"/>
-<wire x1="10.4064" y1="45.75" x2="12" y2="45.75" width="0.2" layer="1"/>
-<wire x1="10" y1="47" x2="10" y2="45.3436" width="0.2" layer="16"/>
+<via x="10" y="45" extent="1-16" drill="0.3"/>
+<wire x1="10" y1="47" x2="10" y2="45" width="0.2" layer="16"/>
 <contactref element="J1" pad="A7"/>
 <contactref element="J1" pad="B7"/>
@@
 <wire x1="6.5" y1="46" x2="6.75" y2="45.75" width="0.2" layer="1"/>
 <wire x1="6.75" y1="45.75" x2="7.5" y2="45.75" width="0.2" layer="1"/>
+<wire x1="10.75" y1="45.75" x2="12" y2="45.75" width="0.2" layer="1"/>
+<wire x1="10" y1="45" x2="10.75" y2="45.75" width="0.2" layer="1"/>
 </signal>
 <signal name="RTS">
