File: blimp/pcb/blimpy-2.0.sch (EAGLE design)
At the start: 153 parts, among them J1 MICRO-USB, J10 3-PIN SMD, J11 3-PIN SMD, J12 3-PIN SMD, J13 3-PIN SMD, J14 3-PIN SMD, J9 3-PIN SMD, M0 DRV8833PWPR, M1 DRV8833PWPR, M2 DRV8833PWPR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

Commit message: Added LED connector
Parts:
- added J15: 3-PIN SMD, SparkFun-Connectors:CONN_03JST-SMD
- added LED3: VUSB, led:LEDCHIP-LED0603
- added R37: (no value), SparkFun-Resistors:RESISTOR0603
- LED1: value (none) -> 3.3V
- LED2: value (none) -> VBAT
Connections:
- removed net LEDRING: TP5.1, U9.14-IO
- new net LEDEXT: J15.2, TP5.1, U9.14-IO
- new net N$17: LED3.C, R37.1
- net 3.3V: now also J15.3
- net GND: now also J15.1, R37.2
- net V_USB: now also LED3.A
Other:
- moved on the sheet: C13, C15, C21

Commit message: Cosmetic changes
Parts:
- Q1, Q2: value mmbt2222 -> 600mA/40V; device SparkFun:TRANSISTOR_NPNSOT23-3 -> SparkFun-DiscreteSemi:TRANS_NPN-MMBT2222AL
- R3: value 0.05 -> 0.005
Changed lines of the file:
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@@
 <part name="U7" library="microbuilder" deviceset="CP2104" device="" value="CP2104"/>
 <part name="C2" library="SparkFun-Capacitors" deviceset="10UF" device="-0603-6.3V-20%" package3d_urn="urn:adsk.eagle:package:37414/1" value="10uF"/>
-<part name="Q1" library="SparkFun" deviceset="TRANSISTOR_NPN" device="SOT23-3" value="mmbt2222"/>
-<part name="Q2" library="SparkFun" deviceset="TRANSISTOR_NPN" device="SOT23-3" value="mmbt2222"/>
 <part name="Q3" library="microbuilder" deviceset="MOSFET-P" device="" value="DMG3415U"/>
 <part name="R12" library="SparkFun-Resistors" deviceset="100KOHM" device="-0603-1/10W-1%" value="100k"/>
@@
 <part name="R1" library="SparkFun-Resistors" library_urn="urn:adsk.eagle:library:532" deviceset="10OHM" device="-0603-1/10W-1%" package3d_urn="urn:adsk.eagle:package:39650/1" value="10"/>
 <part name="C1" library="SparkFun-Capacitors" deviceset="470NF" device="-0608" package3d_urn="urn:adsk.eagle:package:37414/1" value="470nF"/>
-<part name="R3" library="SparkFun-Resistors" library_urn="urn:adsk.eagle:library:532" deviceset="RESISTOR" device="1206" package3d_urn="urn:adsk.eagle:package:39654/1" value="0.05"/>
+<part name="R3" library="SparkFun-Resistors" library_urn="urn:adsk.eagle:library:532" deviceset="RESISTOR" device="1206" package3d_urn="urn:adsk.eagle:package:39654/1" value="0.005"/>
 <part name="SUPPLY8" library="SparkFun-PowerSymbols" library_urn="urn:adsk.eagle:library:530" deviceset="V_BATT" device="" value="VBAT"/>
 <part name="J3" library="SparkFun-Connectors" library_urn="urn:adsk.eagle:library:513" deviceset="CONN_02" device="-JST-2MM-SMT" package3d_urn="urn:adsk.eagle:package:38042/1"/>
@@
 <part name="GND45" library="SparkFun-PowerSymbols" library_urn="urn:adsk.eagle:library:530" deviceset="GND" device=""/>
 <part name="SUPPLY32" library="SparkFun-PowerSymbols" library_urn="urn:adsk.eagle:library:530" deviceset="3.3V" device=""/>
+<part name="Q2" library="SparkFun-DiscreteSemi" library_urn="urn:adsk.eagle:library:514" deviceset="TRANS_NPN" device="-MMBT2222AL" package3d_urn="urn:adsk.eagle:package:38446/1" value="600mA/40V"/>
+<part name="Q1" library="SparkFun-DiscreteSemi" library_urn="urn:adsk.eagle:library:514" deviceset="TRANS_NPN" device="-MMBT2222AL" package3d_urn="urn:adsk.eagle:package:38446/1" value="600mA/40V"/>
 </parts>
 <sheets>
@@
 <attribute name="NAME" x="378.46" y="128.27" size="1.778" layer="95"/>
 </instance>
-<instance part="Q1" gate="G$1" x="208.28" y="-12.7" smashed="yes" rot="MR180">
-<attribute name="NAME" x="213.36" y="-12.7" size="1.778" layer="95" rot="MR180"/>
-<attribute name="VALUE" x="213.36" y="-10.16" size="1.778" layer="96" rot="MR180"/>
-</instance>
-<instance part="Q2" gate="G$1" x="208.28" y="5.08" smashed="yes">
-<attribute name="NAME" x="213.36" y="5.08" size="1.778" layer="95"/>
-<attribute name="VALUE" x="213.36" y="2.54" size="1.778" layer="96"/>
-</instance>
 <instance part="Q3" gate="G$1" x="182.88" y="200.66" smashed="yes" rot="MR180">
 <attribute name="VALUE" x="185.674" y="202.565" size="1.27" layer="96" rot="MR180"/>
@@
 <attribute name="VALUE" x="396.24" y="13.716" size="1.27" layer="96" align="bottom-center"/>
 </instance>
+<instance part="Q2" gate="G$1" x="208.28" y="5.08" smashed="yes">
+<attribute name="NAME" x="210.82" y="5.08" size="1.778" layer="95" font="vector"/>
+<attribute name="VALUE" x="210.82" y="2.794" size="1.778" layer="96" font="vector"/>
+</instance>
+<instance part="Q1" gate="G$1" x="208.28" y="-12.7" smashed="yes" rot="MR180">
+<attribute name="NAME" x="210.82" y="-12.7" size="1.778" layer="95" font="vector" rot="MR180"/>
+<attribute name="VALUE" x="210.82" y="-10.414" size="1.778" layer="96" font="vector" rot="MR180"/>
+</instance>
 </instances>
 <busses>
@@
 <wire x1="187.96" y1="5.08" x2="190.5" y2="5.08" width="0.1524" layer="91"/>
 <junction x="187.96" y="5.08"/>
-<pinref part="Q1" gate="G$1" pin="E"/>
 <wire x1="187.96" y1="5.08" x2="180.34" y2="5.08" width="0.1524" layer="91"/>
 <label x="180.34" y="5.08" size="1.27" layer="95" rot="MR0" xref="yes"/>
 <pinref part="R9" gate="G$1" pin="1"/>
+<pinref part="Q1" gate="G$1" pin="E"/>
 </segment>
 </net>
@@
 <wire x1="187.96" y1="-12.7" x2="190.5" y2="-12.7" width="0.1524" layer="91"/>
 <junction x="187.96" y="-12.7"/>
-<pinref part="Q2" gate="G$1" pin="E"/>
 <wire x1="187.96" y1="-12.7" x2="180.34" y2="-12.7" width="0.1524" layer="91"/>
 <label x="180.34" y="-12.7" size="1.27" layer="95" rot="MR0" xref="yes"/>
 <pinref part="R10" gate="G$1" pin="1"/>
+<pinref part="Q2" gate="G$1" pin="E"/>
 </segment>
 </net>
@@
 <segment>
 <wire x1="205.74" y1="-12.7" x2="200.66" y2="-12.7" width="0.1524" layer="91"/>
+<pinref part="R10" gate="G$1" pin="2"/>
 <pinref part="Q1" gate="G$1" pin="B"/>
-<pinref part="R10" gate="G$1" pin="2"/>
 </segment>
 </net>
@@
 <segment>
 <wire x1="200.66" y1="5.08" x2="205.74" y2="5.08" width="0.1524" layer="91"/>
+<pinref part="R9" gate="G$1" pin="2"/>
 <pinref part="Q2" gate="G$1" pin="B"/>
-<pinref part="R9" gate="G$1" pin="2"/>
 </segment>
 </net>
@@
 <segment>
 <wire x1="210.82" y1="10.16" x2="218.44" y2="10.16" width="0.1524" layer="91"/>
+<label x="218.44" y="10.16" size="1.27" layer="95" xref="yes"/>
 <pinref part="Q2" gate="G$1" pin="C"/>
-<label x="218.44" y="10.16" size="1.27" layer="95" xref="yes"/>
 </segment>
 </net>
@@
 <segment>
 <wire x1="218.44" y1="-17.78" x2="210.82" y2="-17.78" width="0.1524" layer="91"/>
+<label x="218.44" y="-17.78" size="1.27" layer="95" xref="yes"/>
 <pinref part="Q1" gate="G$1" pin="C"/>
-<label x="218.44" y="-17.78" size="1.27" layer="95" xref="yes"/>
-</segment>
-<segment>
+</segment>
+<segment>

Commit message: Motor driver bug fix, added pull-up for btn input, cosmetic changes
Parts:
- removed LED1: 3.3V, led:LEDCHIP-LED0603
- removed LED2: VBAT, led:LEDCHIP-LED0603
- removed LED3: VUSB, led:LEDCHIP-LED0603
- added D4, D5, D6: GREEN, microbuilder:LED0805_NOOUTLINE
- added R38: 4.7k, SparkFun-Resistors:1MOHM-0603-1/4W-5%
- renumbered U$1 to S1
Connections:
- removed net N$20: TP8.1, U9.34-IA
- removed net PWM0-A: J11.3, M0.A_IN1, M0.A_IN2, TP1.1, U9.32-IOA
- removed net PWM0-B: J12.3, M0.B_IN1, M0.B_IN2, TP2.1, U9.33-IOA
- removed net PWM1-A: J13.3, M1.A_IN1, M1.A_IN2, TP3.1, U9.25-IOD
- removed net PWM1-B: J14.3, M1.B_IN1, M1.B_IN2, TP6.1, U9.26-IOD
- removed net PWM2-A: M2.A_IN1, M2.A_IN2, TP17.1, U9.27-IO
- removed net PWM2-B: M2.B_IN1, M2.B_IN2, TP23.1, U9.13-IO
- removed net PWM3-A: M3.A_IN1, M3.A_IN2, TP16.1, U9.4-IO
- removed net PWM3-B: M3.B_IN1, M3.B_IN2, TP15.1, U9.16-IO
- removed net PWM4-A: M4.A_IN1, M4.A_IN2, TP22.1, U9.17-IO
- removed net PWM4-B: M4.B_IN1, M4.B_IN2, TP21.1, U9.18-IO
- removed net PWM5-A: M5.A_IN1, M5.A_IN2, TP20.1, U9.19-IO
- removed net PWM5-B: M5.B_IN1, M5.B_IN2, TP14.1, U9.23-IO
- new net N$58: J3.2, M0.A_OUT2, M0.B_OUT2
- new net PWM0-1: J11.3, M0.A_IN1, M0.B_IN1, TP1.1, U9.32-IOA
- new net PWM0-2: J12.3, M0.A_IN2, M0.B_IN2, TP2.1, U9.33-IOA
- new net PWM1-1: J13.3, M1.A_IN1, M1.B_IN1, TP3.1, U9.25-IOD
- new net PWM1-2: J14.3, M1.A_IN2, M1.B_IN2, TP6.1, U9.26-IOD
- new net PWM2-1: M2.A_IN1, M2.B_IN1, TP17.1, U9.27-IO
- new net PWM2-2: M2.A_IN2, M2.B_IN2, TP23.1, U9.13-IO
- new net PWM3-1: M3.A_IN1, M3.B_IN1, TP16.1, U9.4-IO
- new net PWM3-2: M3.A_IN2, M3.B_IN2, TP15.1, U9.16-IO
- new net PWM4-1: M4.A_IN1, M4.B_IN1, TP22.1, U9.17-IO
- new net PWM4-2: M4.A_IN2, M4.B_IN2, TP21.1, U9.18-IO
- new net PWM5-1: M5.A_IN1, M5.B_IN1, TP20.1, U9.19-IO
- new net PWM5-2: M5.A_IN2, M5.B_IN2, TP14.1, U9.23-IO
- net 3.3V: now also D6.A, R38.2; no longer LED1.A
- net BTN: now also R38.1, TP8.1, U9.34-IA; no longer TP10.1, U9.36-I
- net N$17: now also D4.C; no longer LED3.C
- net N$24: now also J4.2, M1.B_OUT2; no longer J4.1, M1.A_OUT1
- net N$25: now also J4.1, M1.A_OUT1; no longer J4.2, M1.B_OUT2
- net N$30: now also J6.2, M3.A_OUT2, M3.B_OUT2; no longer J5.1, M2.A_OUT1, M2.A_OUT2
- net N$31: now also M2.A_OUT2; no longer M2.B_OUT1
- net N$36: now also M3.B_OUT1; no longer M3.A_OUT2
- net N$37: now also M0.B_OUT1; no longer M0.A_OUT2
- net N$38: now also J7.2, M4.A_OUT2, M4.B_OUT2; no longer J6.2, M3.B_OUT1, M3.B_OUT2
- net N$43: now also J8.1, M5.A_OUT1, M5.B_OUT1; no longer J7.1, M4.A_OUT1, M4.A_OUT2
- net N$44: now also J7.1, M4.A_OUT1; no longer J7.2, M4.B_OUT2
- net N$48: now also J5.1, M2.A_OUT1, M2.B_OUT1; no longer J3.2, M0.B_OUT1, M0.B_OUT2
- net N$50: now also J8.2, M5.B_OUT2; no longer J8.1, M5.A_OUT1
- net N$51: now also D6.C, R36.1; no longer J8.2, M5.B_OUT1, M5.B_OUT2
- net N$56: now also D5.C; no longer LED2.C
- net N$57: now also TP10.1, U9.36-I; no longer LED1.C, R36.1
- net V_BATT: now also D5.A; no longer LED2.A
- net V_USB: now also D4.A; no longer LED3.A
Other:
- moved on the sheet: J4, J5, J6, J7, J8

Commit message: Added jumper to disable charging when MC is running
Parts:
- added JP2: JUMPER-SMT_2_NO_SILK, SparkFun-Jumpers:JUMPER-SMT_2_NO_SILK
Connections:
- net N$4: now also JP2.1
- net PWR: now also JP2.2
Changed lines of the file:
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@@
 <part name="R38" library="SparkFun-Resistors" library_urn="urn:adsk.eagle:library:532" deviceset="1MOHM" device="-0603-1/4W-5%" package3d_urn="urn:adsk.eagle:package:39650/1" value="4.7k"/>
 <part name="SUPPLY33" library="SparkFun-PowerSymbols" library_urn="urn:adsk.eagle:library:530" deviceset="3.3V" device=""/>
+<part name="JP2" library="SparkFun-Jumpers" library_urn="urn:adsk.eagle:library:528" deviceset="JUMPER-SMT_2_NO" device="_SILK" package3d_urn="urn:adsk.eagle:package:39279/1"/>
 </parts>
 <sheets>
@@
 <attribute name="VALUE" x="43.18" y="191.516" size="1.27" layer="96" align="bottom-center"/>
 </instance>
+<instance part="JP2" gate="G$1" x="375.92" y="205.74" smashed="yes" rot="R90">
+<attribute name="NAME" x="373.38" y="203.2" size="1.778" layer="95" font="vector" rot="R90"/>
+</instance>
 </instances>
 <busses>
@@
 <junction x="368.3" y="195.58"/>
 <pinref part="U3" gate="G$1" pin="PROG"/>
+<pinref part="JP2" gate="G$1" pin="1"/>
+<wire x1="368.3" y1="195.58" x2="375.92" y2="195.58" width="0.1524" layer="91"/>
+<wire x1="375.92" y1="195.58" x2="375.92" y2="200.66" width="0.1524" layer="91"/>
 </segment>
 </net>
@@
 <label x="167.64" y="86.36" size="1.27" layer="95"/>
 </segment>
-</net>
+<segment>
+<pinref part="JP2" gate="G$1" pin="2"/>
+<wire x1="375.92" y1="210.82" x2="375.92" y2="218.44" width="0.1524" layer="91"/>
+<label x="375.92" y="218.44" size="1.27" layer="95" rot="R90" xref="yes"/>
+</segment>
+</net>
