File: blimp/pcb/blimpy-2.1.brd (EAGLE design)
At the start: 80 x 70 mm, 154 parts, among them J1 MICRO-USB, J10 3-PIN SMD, J11 3-PIN SMD, J12 3-PIN SMD, J13 3-PIN SMD, J14 3-PIN SMD, J15 3-PIN SMD, J9 3-PIN SMD, M0 DRV8833PWPR, M1 DRV8833PWPR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

Commit message: PCB 2.1 production
Parts:
- added JP2: JUMPER-SMT_2_NO_SILK, SparkFun-Jumpers:SMT-JUMPER_2_NO_SILK
Connections:
- new net N$20: D1.A, JP2.1, Q3.1, R12.2
- net V_USB: now also JP2.2; no longer D1.A, Q3.1, R12.2
Routing:
- net N$20: track 0.00 -> 16.5 mm
- net V_USB: track 79.0 -> 71.8 mm
Changed lines of the file:
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@@
 <attribute name="PROD_ID" value="RES-07868" x="62.4" y="48.3" size="1.778" layer="27" rot="R90" display="off"/>
+</element>
+<element name="JP2" library="SparkFun-Jumpers" library_urn="urn:adsk.eagle:library:528" package="SMT-JUMPER_2_NO_SILK" package3d_urn="urn:adsk.eagle:package:39279/1" value="JUMPER-SMT_2_NO_SILK" x="39.1" y="32.6" smashed="yes">
+<attribute name="NAME" x="39.1" y="33.743" size="0.6" layer="25" font="vector" ratio="20" align="bottom-center"/>
 </element>
 </elements>
@@
 <contactref element="D2" pad="A"/>
 <contactref element="C9" pad="1"/>
-<contactref element="R12" pad="2"/>
-<contactref element="D1" pad="A"/>
-<contactref element="Q3" pad="1"/>
 <contactref element="JP1" pad="2"/>
 <contactref element="J1" pad="VBUS"/>
@@
 <wire x1="45.2" y1="17.1" x2="45.2" y2="17.9501" width="0.2" layer="1"/>
 <wire x1="45.2" y1="17.9501" x2="45.15" y2="18.0001" width="0.2" layer="1"/>
-<wire x1="33.25" y1="32.6" x2="34.75" y2="32.6" width="0.2" layer="1"/>
 <via x="60.7436" y="14.18469375" extent="1-16" drill="0.3"/>
 <wire x1="60.7436" y1="14.18469375" x2="61.0476" y2="13.88069375" width="0.2" layer="1"/>
@@
 <wire x1="61.0476" y1="13.84645625" x2="61.34405625" y2="13.55" width="0.2" layer="1"/>
 <wire x1="61.34405625" y1="13.55" x2="61.7" y2="13.55" width="0.2" layer="1"/>
-<wire x1="34.75" y1="32.6" x2="35.95" y2="33.8" width="0.2" layer="1"/>
-<wire x1="35.95" y1="33.8" x2="37.1" y2="33.8" width="0.2" layer="1"/>
 <wire x1="46.85" y1="18.1" x2="46.85" y2="15.45" width="0.2" layer="1"/>
 <wire x1="46.85" y1="15.45" x2="47" y2="15.3" width="0.2" layer="1"/>
@@
 <wire x1="74.09109375" y1="14.18469375" x2="75.55" y2="15.6436" width="0.2" layer="16"/>
 <via x="75.55" y="15.6436" extent="1-16" drill="0.3"/>
-<wire x1="37.5" y1="38.45" x2="36.75" y2="39.2" width="0.2" layer="1"/>
-<wire x1="37.1" y1="33.8" x2="37.5" y2="34.2" width="0.2" layer="1"/>
-<wire x1="37.5" y1="34.2" x2="37.5" y2="38.45" width="0.2" layer="1"/>
 <wire x1="46.85" y1="18.1" x2="46.85" y2="19.2564" width="0.2" layer="1"/>
 <wire x1="46.85" y1="19.2564" x2="44.5064" y2="21.6" width="0.2" layer="1"/>
 <contactref element="D4" pad="A"/>
-<wire x1="41" y1="25.3" x2="41" y2="17.75" width="0.2" layer="1"/>
-<wire x1="36.75" y1="39.2" x2="37.75" y2="39.2" width="0.2" layer="1"/>
-<wire x1="37.75" y1="39.2" x2="39.4" y2="40.85" width="0.2" layer="1"/>
-<wire x1="34.75" y1="32.6" x2="34.75" y2="31.65" width="0.2" layer="1"/>
-<wire x1="41" y1="25.4" x2="41" y2="25.3" width="0.2" layer="1"/>
-<wire x1="34.75" y1="31.65" x2="41" y2="25.4" width="0.2" layer="1"/>
+<wire x1="41" y1="31.1064" x2="41" y2="17.75" width="0.2" layer="1"/>
+<contactref element="JP2" pad="2"/>
+<wire x1="39.4" y1="40.85" x2="39.4" y2="32.7064" width="0.2" layer="1"/>
+<wire x1="39.4" y1="32.7064" x2="39.5064" y2="32.6" width="0.2" layer="1"/>
+<wire x1="39.5064" y1="32.6" x2="41" y2="31.1064" width="0.2" layer="1"/>
 </signal>
 <signal name="V_BATT">
@@
 <wire x1="64.89" y1="45.977309375" x2="64.89" y2="44" width="0.2" layer="1"/>
 </signal>
+<signal name="N$20">
+<contactref element="R12" pad="2"/>
+<contactref element="D1" pad="A"/>
+<contactref element="Q3" pad="1"/>
+<wire x1="33.25" y1="32.6" x2="34.75" y2="32.6" width="0.2" layer="1"/>
+<wire x1="34.75" y1="32.6" x2="35.95" y2="33.8" width="0.2" layer="1"/>
+<wire x1="35.95" y1="33.8" x2="37.1" y2="33.8" width="0.2" layer="1"/>
+<wire x1="37.5" y1="38.45" x2="36.75" y2="39.2" width="0.2" layer="1"/>
+<wire x1="37.1" y1="33.8" x2="37.5" y2="34.2" width="0.2" layer="1"/>
+<wire x1="37.5" y1="34.2" x2="37.5" y2="38.45" width="0.2" layer="1"/>
+<contactref element="JP2" pad="1"/>
+<wire x1="33.25" y1="32.6" x2="34.25" y2="31.6" width="0.2" layer="1"/>
+<wire x1="37.6936" y1="31.6" x2="38.6936" y2="32.6" width="0.2" layer="1"/>
+<wire x1="34.25" y1="31.6" x2="37.6936" y2="31.6" width="0.2" layer="1"/>
+</signal>
 </signals>
