File: robots/blimpy/design/electronics/pcb/blimpy-2.1.sch (EAGLE design)
At the start: 155 parts, among them J1 MICRO-USB, J10 3-PIN SMD, J11 3-PIN SMD, J12 3-PIN SMD, J13 3-PIN SMD, J14 3-PIN SMD, J15 3-PIN SMD, J9 3-PIN SMD, M0 DRV8833PWPR, M1 DRV8833PWPR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

Commit message: Restructured directories to accommodate different hardware platforms
Other:
- note added: "Blimpy Board 2.1 Immersive Arts Space ZHdK - Joël Gähwiler, Max Kriegleder"
- note removed: "Blimpy Board 2.0 Immersive Arts Space ZHdK - Joël Gähwiler, Max Kriegleder"
Changed lines of the file:
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@@
 <text x="680.72" y="220.98" size="1.778" layer="94">SERVOS</text>
 <text x="449.58" y="223.52" size="1.778" layer="94">MOTORS</text>
-<text x="10.16" y="-58.42" size="6.35" layer="95">Blimpy Board 2.0
+<text x="10.16" y="-58.42" size="6.35" layer="95">Blimpy Board 2.1
 Immersive Arts Space
 ZHdK - Joël Gähwiler, Max Kriegleder</text>
